File: power_switch.kicad_pcb (KiCad board)
At the start: 2 copper layers, 110 parts, among them IC1 ATTINY2313A-P, P1 CONN_2, P10 CONN_01X01, P11 CONN_02X01, P12 CONN_01X01, P13 CONN_2, P14 CONN_2, P15 CONN_2, P16 CONN_2, P17 CONN_2, P18 CONN_2, P19 CONN_2, P2 CONN_2, P20 CONN_2, P21 CONN_01X03, P3 CONN_2, P4 CONN_2, P5 CONN_2, P6 CONN_01X03, P7 CONN_01X01, P8 CONN_01X01, P9 CONN_01X01, Q1 Q_NPN_EBC, Q10 Q_NJFET_DGS, Q11 Q_NPN_EBC, Q12 Q_NPN_EBC, Q13 Q_NJFET_DGS, Q14 Q_NJFET_DGS, Q2 Q_NJFET_DGS, Q3 Q_NPN_EBC, Q4 Q_NPN_EBC, Q5 Q_NJFET_DGS, Q6 Q_NJFET_DGS, Q7 Q_NPN_EBC, Q8 Q_NPN_EBC, Q9 Q_NJFET_DGS, U1 LTV-817, U2 LTV-817, U3 LTV-817, U4 LTV-817, U5 LTV-817, U6 LM317T, U7 LTV-817, U8 LTV-817, U9 LTV-817

Commit message: initial commit
Parts:
- added P22: CONN_01X09, Socket_Strips:Socket_Strip_Straight_1x09, F.Cu at (331.5, 50.8)
- added P23: CONN_01X09, Socket_Strips:Socket_Strip_Straight_1x08, F.Cu at (381.0, 137.2)
- added R32: 150R, Resistors_ThroughHole:Resistor_Horizontal_RM7mm, F.Cu at (309.9, 5.08)
- added R33: 150R, Resistors_ThroughHole:Resistor_Horizontal_RM7mm, F.Cu at (334.0, -11.4)
- added R34: 150R, Resistors_ThroughHole:Resistor_Horizontal_RM7mm, F.Cu at (346.7, -12.7)
- added R35: 150R, Resistors_ThroughHole:Resistor_Horizontal_RM7mm, F.Cu at (365.8, -12.7)
- added R36: 150R, Resistors_ThroughHole:Resistor_Horizontal_RM7mm, F.Cu at (378.5, -12.7)
- added R37: 150R, Resistors_ThroughHole:Resistor_Horizontal_RM7mm, F.Cu at (395.0, -12.7)
- added R38: 150R, Resistors_ThroughHole:Resistor_Horizontal_RM7mm, F.Cu at (420.4, -12.7)
- added R39: 150R, Resistors_ThroughHole:Resistor_Horizontal_RM7mm, F.Cu at (435.6, -11.4)
- C4: value 4.7uF -> 47uf
- moved R22 139.1 mm to (222.2, 85.1)
- moved U1 126.9 mm to (337.8, 110.5)
- moved U2 126.9 mm to (363.2, 110.5)
- moved U3 126.9 mm to (378.5, 110.5)
- moved U4 126.9 mm to (393.7, 110.5)
- moved U5 126.9 mm to (407.7, 110.5)
- moved U7 126.9 mm to (422.9, 110.5)
- moved U8 126.9 mm to (453.4, 110.5)
- moved U9 126.9 mm to (473.7, 110.5)
- moved R7 118.1 mm to (228.6, 134.6)
- moved R9 117.3 mm to (416.6, 83.8)
- moved R1 107.7 mm to (388.6, 73.7)
- moved JP2 100.1 mm to (395.0, 5.08), turned to 270 degrees
- moved JP6 97.7 mm to (298.4, 0.00)
- moved R11 92.9 mm to (419.1, 62.2)
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Connections:
- 2k1 pad 2: +3V3 -> (no net)
- C4 pad 1: +9V -> +3V3
- IC1 pad 11: /ts1 -> /ts7
- IC1 pad 12: /ts8 -> Net-(D15-Pad2)
- IC1 pad 13: /sw_E -> Net-(D14-Pad2)
- IC1 pad 14: /sw_T -> Net-(D13-Pad2)
- IC1 pad 15: /sw_R -> Net-(D10-Pad2)
- IC1 pad 16: /sw_V -> Net-(D9-Pad2)
- IC1 pad 17: /sw_U -> Net-(D6-Pad2)
- IC1 pad 18: /sw_Y -> Net-(D5-Pad2)
- IC1 pad 19: /sw_X -> Net-(D1-Pad2)
- IC1 pad 2: /ts7 -> /ts1
- IC1 pad 3: /ts6 -> /ts2
- IC1 pad 4: /ts10 -> /ts9
- IC1 pad 5: /ts9 -> /ts8
- IC1 pad 6: /ts5 -> /ts3
- IC1 pad 8: /ts3 -> /ts5
- IC1 pad 9: /ts2 -> /ts6
- P10 pad 1: Net-(P10-Pad1) -> (no net)
- P12 pad 1: Net-(P12-Pad1) -> (no net)
- P6 pad 1: /sw_X -> Net-(D1-Pad2)
- P6 pad 2: /sw_Y -> Net-(D5-Pad2)
- P6 pad 3: /sw_U -> Net-(D6-Pad2)
- P7 pad 1: Net-(P7-Pad1) -> (no net)
- P9 pad 1: Net-(P9-Pad1) -> (no net)
- R1 pad 2: Net-(D1-Pad1) -> Net-(R1-Pad2)
- R11 pad 2: Net-(D6-Pad1) -> Net-(R11-Pad2)
- R18 pad 2: Net-(D9-Pad1) -> Net-(R18-Pad2)
- R20 pad 2: Net-(D10-Pad1) -> Net-(R20-Pad2)
- R26 pad 2: Net-(D13-Pad1) -> Net-(R26-Pad2)
- R28 pad 2: Net-(D14-Pad1) -> Net-(R28-Pad2)
- R31 pad 2: Net-(D15-Pad1) -> Net-(R31-Pad2)
- R9 pad 2: Net-(D5-Pad1) -> Net-(R9-Pad2)
- U1 pad 1: /sw_X -> (no net)
- U1 pad 2: Net-(D1-Pad2) -> Net-(R1-Pad2)
- U2 pad 2: Net-(D5-Pad2) -> Net-(R9-Pad2)
- U3 pad 2: Net-(D6-Pad2) -> Net-(R11-Pad2)
- U4 pad 2: Net-(D9-Pad2) -> Net-(R18-Pad2)
- U5 pad 2: Net-(D10-Pad2) -> Net-(R20-Pad2)
- U7 pad 2: Net-(D13-Pad2) -> Net-(R26-Pad2)
- U8 pad 2: Net-(D14-Pad2) -> Net-(R28-Pad2)
- U9 pad 2: Net-(D15-Pad2) -> Net-(R31-Pad2)
Routing:
- net /ts1: track 0.00 -> 92.9 mm
- net (no net): track 0.00 -> 78.1 mm
- net /ts2: track 0.00 -> 67.3 mm
- net /ts6: track 0.00 -> 56.2 mm
- net /ts9: track 0.00 -> 55.9 mm
- net /ts8: track 0.00 -> 43.4 mm
- net /ts5: track 0.00 -> 37.8 mm
- net /ts3: track 0.00 -> 32.7 mm
- net /ts4: track 0.00 -> 29.8 mm
- net /sw_Y: track 3.81 -> 0.00 mm
- net /sw_X: track 3.81 -> 0.00 mm
- net /sw_U: track 3.81 -> 0.00 mm
- net Net-(IC1-Pad1): track 6.35 -> 7.62 mm
- net Net-(D15-Pad2): track 10.5 -> 11.2 mm
- net Net-(D9-Pad2): track 10.5 -> 11.2 mm
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
Commit message: simplified version
Parts:
- moved JP5 12.3 mm to (319.4, 11.4)
- moved JP1 11.5 mm to (408.9, 5.08)
- moved U1 0.90 mm to (337.2, 111.1)
- moved D9 0.12 mm to (365.1, 0.00)
Routing:
- net /ts1: track 92.9 -> 81.6 mm
- net /ts5: track 37.8 -> 27.8 mm
Changed lines of the file:
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@@
     (links 234)
     (no_connects 199)
-    (area 0 0 0 0)
+    (area 163.576667 -17.47512 479.235001 187.96012)
     (thickness 1.6)
     (drawings 0)
@@
   )
   (module LEDs:LED-3MM (layer F.Cu)
-    (at 365 0 90)
+    (at 365.125 0 90)
     (descr "LED 3mm round vertical")
     (tags "LED  3mm round vertical")
@@
   )
   (module Buttons_Switches_ThroughHole:SW_PUSH_6mm (layer F.Cu)
-    (at 410.21 -6.35 270)
+    (at 408.94 5.08 270)
     (descr https://www.omron.com/ecb/products/pdf/en-b3f.pdf)
     (tags "tact sw push 6mm")
@@
   )
   (module Buttons_Switches_ThroughHole:SW_PUSH_6mm (layer F.Cu)
-    (at 323.85 0 90)
+    (at 319.405 11.43 90)
     (descr https://www.omron.com/ecb/products/pdf/en-b3f.pdf)
     (tags "tact sw push 6mm")
@@
   )
   (module Housings_DIP:DIP-4_W7.62mm_LongPads (layer F.Cu)
-    (at 337.82 110.49 90)
+    (at 337.185 111.125 90)
     (descr "4-lead dip package, row spacing 7.62 mm (300 mils), longer pads")
     (tags "dil dip 2.54 300")
@@
   (segment (start 346.71 22.86) (end 346.71 33.02) (width 1) (layer F.Cu) (net 13))
   (segment (start 376.5 11.58) (end 376.5 5.08) (width 1) (layer F.Cu) (net 13))
-  (segment (start 328.35 -6.5) (end 328.35 0) (width 1) (layer F.Cu) (net 14))
+  (segment (start 323.905 4.93) (end 323.905 11.43) (width 1) (layer F.Cu) (net 14) (status 30))
   (segment (start 336.55 33.02) (end 336.55 30.898676) (width 1) (layer F.Cu) (net 14))
-  (segment (start 328.35 17.618676) (end 328.35 0) (width 1) (layer F.Cu) (net 14))
+  (segment (start 328.35 17.618676) (end 323.905 11.43) (width 1) (layer F.Cu) (net 14) (status 20))
   (segment (start 336.55 30.898676) (end 328.35 22.698676) (width 1) (layer F.Cu) (net 14))
   (segment (start 339.09 17.78) (end 339.09 16.51) (width 1) (layer F.Cu) (net 15))
-  (segment (start 339.09 16.51) (end 339.09 12.01) (width 1) (layer F.Cu) (net 15) (status 800000))
-  (segment (start 338.51 4.93) (end 338.51 11.43) (width 1) (layer F.Cu) (net 15) (status C00000))
-  (segment (start 338.51 11.43) (end 339.09 12.01) (width 1) (layer F.Cu) (net 15) (status C00000))
+  (segment (start 339.09 16.51) (end 339.09 12.01) (width 1) (layer F.Cu) (net 15))
+  (segment (start 338.51 4.93) (end 338.51 11.43) (width 1) (layer F.Cu) (net 15))
+  (segment (start 338.51 11.43) (end 339.09 12.01) (width 1) (layer F.Cu) (net 15))
   (segment (start 339.09 33.02) (end 339.09 17.78) (width 1) (layer F.Cu) (net 15) (status 20))
   (segment (start 339.09 17.78) (end 339.09 17.09) (width 1) (layer F.Cu) (net 15) (status 20))
@@
   (segment (start 341.63 20.32) (end 341.63 33.02) (width 1) (layer F.Cu) (net 16))
   (segment (start 348.56 11.58) (end 348.56 5.08) (width 1) (layer F.Cu) (net 16))
-  (segment (start 349.25 33.02) (end 349.25 27.94) (width 1) (layer F.Cu) (net 17) (status 400000))
+  (segment (start 349.25 33.02) (end 349.25 27.94) (width 1) (layer F.Cu) (net 17))
   (segment (start 349.25 20.32) (end 350.52 19.05) (width 1) (layer F.Cu) (net 17))
   (segment (start 350.52 19.05) (end 388.62 19.05) (width 1) (layer F.Cu) (net 17))
@@
   (segment (start 351.79 22.86) (end 353.06 21.59) (width 1) (layer F.Cu) (net 18))
   (segment (start 351.79 33.02) (end 351.79 22.86) (width 1) (layer F.Cu) (net 18))
-  (segment (start 405.71 19.74) (end 405.71 0.15) (width 1) (layer F.Cu) (net 18) (status 800000))
+  (segment (start 405.71 19.74) (end 404.44 11.58) (width 1) (layer F.Cu) (net 18) (status 20))
   (segment (start 403.86 21.59) (end 405.71 19.74) (width 1) (layer F.Cu) (net 18))
   (segment (start 353.06 21.59) (end 403.86 21.59) (width 1) (layer F.Cu) (net 18))
-  (segment (start 405.71 -6.35) (end 405.71 0.15) (width 1) (layer F.Cu) (net 18))
-  (segment (start 405.71 0.15) (end 405.86 0) (width 1) (layer F.Cu) (net 18))
-  (segment (start 405.86 0) (end 406.4 0) (width 1) (layer F.Cu) (net 18))
-  (segment (start 406.4 0) (end 405.71 0.15) (width 1) (layer F.Cu) (net 18))
+  (segment (start 404.44 5.08) (end 404.44 11.58) (width 1) (layer F.Cu) (net 18) (status 30))
+  (segment (start 404.44 11.58) (end 404.59 11.43) (width 1) (layer F.Cu) (net 18) (status 30))
+  (segment (start 404.59 11.43) (end 405.13 11.43) (width 1) (layer F.Cu) (net 18) (status 30))
+  (segment (start 405.13 11.43) (end 404.44 11.58) (width 1) (layer F.Cu) (net 18) (status 30))
   (segment (start 344.17 16.51) (end 344.17 21.59) (width 1) (layer F.Cu) (net 19))
   (segment (start 362.53 11.58) (end 360.14 13.97) (width 1) (layer F.Cu) (net 19))

Commit message: versin with buck converter for amp meter backup
Parts:
- removed 1k1, 2k1: R, Resistors_ThroughHole:Resistor_Horizontal_RM7mm
- removed D10, D13, D14, D15, D9: Led_Small, LEDs:LED-3MM
- removed D11, D12, D8: D, Diodes_ThroughHole:Diode_DO-35_SOD27_Horizontal_RM10
- removed IC1: ATTINY2313A-P, Housings_DIP:DIP-20_W7.62mm_LongPads
- removed JP10, JP3, JP4, JP5, JP6, JP7, JP8, JP9: Jumper_NO_Small, Buttons_Switches_ThroughHole:SW_PUSH_6mm
- removed P14, P15, P16, P17, P18, P19: CONN_2, borniers:bornier2_V
- removed P21: CONN_01X03, Pin_Headers:Pin_Header_Straight_1x03
- removed P22: CONN_01X09, Socket_Strips:Socket_Strip_Straight_1x09
- removed P23: CONN_01X09, Socket_Strips:Socket_Strip_Straight_1x08
- removed Q10, Q13, Q14, Q9: Q_NJFET_DGS, TO_SOT_Packages_THT:TO-220_Neutral123_Vertical_LargePads
- removed Q11, Q12, Q7, Q8: Q_NPN_EBC, TO_SOT_Packages_THT:TO-92_Inline_Narrow_Oval
- removed R20, R26, R28, R31, R32, R33, R34, R35, R36, R37, R38, R39: 150R, Resistors_ThroughHole:Resistor_Horizontal_RM7mm
- removed R21, R27, R29: 20k, Resistors_ThroughHole:Resistor_Horizontal_RM7mm
- removed R22, R24, R30: 100k, Resistors_ThroughHole:Resistor_Horizontal_RM7mm
- removed R23, R25: 68k, Resistors_ThroughHole:Resistor_Horizontal_RM7mm
- removed U2, U3, U4, U5, U7, U8, U9: LTV-817, Housings_DIP:DIP-4_W7.62mm_LongPads
- removed U6: LM317T, Power_Integrations:TO-220
- added C10: 100n, Capacitors_ThroughHole:C_Disc_D3_P2.5, F.Cu at (137.2, 71.1)
- added C11: 10uF, Capacitors_ThroughHole:C_Radial_D8_L13_P3.8, F.Cu at (166.4, 90.2)
- added C12: 100n, Capacitors_ThroughHole:C_Disc_D3_P2.5, F.Cu at (125.7, 77.5)
- added C13: C, Capacitors_ThroughHole:C_Disc_D3_P2.5, F.Cu at (149.9, 63.5)
- added C14: 10uF, Capacitors_ThroughHole:C_Radial_D8_L11.5_P3.5, F.Cu at (193.0, 35.6)
- added C15: 10uF, Capacitors_ThroughHole:C_Radial_D8_L11.5_P3.5, F.Cu at (163.8, 48.3)
- added C16: 10uF, Capacitors_ThroughHole:C_Radial_D8_L11.5_P3.5, F.Cu at (153.7, 48.3)
- added C17: 10uF, Capacitors_ThroughHole:C_Radial_D8_L11.5_P3.5, F.Cu at (174.0, 48.3)
- added C18: 100n, Capacitors_ThroughHole:C_Disc_D3_P2.5, F.Cu at (174.0, 59.7)
- added C8: 10uF, Capacitors_ThroughHole:C_Radial_D10_L20_P7.5, F.Cu at (141.0, 55.9)
- added C9: 100n, Capacitors_ThroughHole:C_Disc_D3_P2.5, F.Cu at (143.5, 92.7)
- added L1: 50uH, Choke_Axial_ThroughHole:Choke_Horizontal_RM10mm, F.Cu at (168.9, 88.9)
- added RV1: POT, Potentiometers:Potentiometer_Bourns_3296X_3-8Zoll_Inline_ScrewFront, F.Cu at (125.7, 67.3)
- C1: value 100n -> 10uF; footprint Capacitors_ThroughHole:C_Disc_D3_P2.5 -> Capacitors_ThroughHole:C_Radial_D10_L20_P7.5
- C2: value 4.7u -> 10uF; footprint Capacitors_ThroughHole:C_Radial_D5_L11_P2 -> Capacitors_ThroughHole:C_Radial_D10_L20_P7.5
- C3, C5: value C_Small -> 10uF; footprint Capacitors_ThroughHole:C_Disc_D3_P2.5 -> Capacitors_ThroughHole:C_Radial_D10_L20_P7.5
- C4: value 47uf -> 10uF; footprint Capacitors_ThroughHole:C_Radial_D5_L11_P2 -> Capacitors_ThroughHole:C_Radial_D10_L20_P7.5
- C6: value 4.7uF -> 10uF; footprint Capacitors_ThroughHole:C_Radial_D5_L11_P2 -> Capacitors_ThroughHole:C_Radial_D10_L20_P7.5
- C7: value 220uF -> 100n; footprint Capacitors_ThroughHole:C_Radial_D5_L11_P2 -> Capacitors_ThroughHole:C_Disc_D3_P2.5
- D1, D5: value Led_Small -> D; footprint LEDs:LED-3MM -> Diodes_ThroughHole:Diode_DO-35_SOD27_Horizontal_RM10
- D6: value Led_Small -> 5v6; footprint LEDs:LED-3MM -> Diodes_ThroughHole:Diode_DO-35_SOD27_Horizontal_RM10
- D7: value D -> 1N4001
- JP1, JP2: footprint Buttons_Switches_ThroughHole:SW_PUSH_6mm -> Pin_Headers:Pin_Header_Angled_1x02_Pitch1.27mm
- P10, P12, P9: value CONN_01X01 -> CONN_2; footprint Mounting_Holes:MountingHole_3.2mm_M3_Pad -> borniers:bornier2_V
- P11: value CONN_02X01 -> CONN_2; footprint Pin_Headers:Pin_Header_Straight_1x02 -> borniers:bornier2_V
- P13: value CONN_2 -> CONN_02X01; footprint borniers:bornier2_V -> Socket_Strips:Socket_Strip_Straight_2x01
- P6: value CONN_01X03 -> CONN_02X01; footprint Pin_Headers:Pin_Header_Straight_1x03 -> Socket_Strips:Socket_Strip_Straight_2x01
- P7: value CONN_01X01 -> CONN_02X01; footprint Mounting_Holes:MountingHole_3.2mm_M3_Pad -> Socket_Strips:Socket_Strip_Straight_2x01
- P8: value CONN_01X01 -> CONN_02X01; footprint Pin_Headers:Pin_Header_Straight_1x01 -> Socket_Strips:Socket_Strip_Straight_2x01
- Q1: value Q_NPN_EBC -> 2N7000; footprint TO_SOT_Packages_THT:TO-92_Inline_Narrow_Oval -> TO_SOT_Packages_THT:TO-220_Neutral123_Vertical_LargePads
- Q2, Q5: value Q_NJFET_DGS -> IRF9540
- Q3: value Q_NPN_EBC -> IRF9540; footprint TO_SOT_Packages_THT:TO-92_Inline_Narrow_Oval -> TO_SOT_Packages_THT:TO-220_Neutral123_Vertical_LargePads
- Q4: value Q_NPN_EBC -> Q_NMOS_DGS
- Q6: value Q_NJFET_DGS -> 2N7000; footprint TO_SOT_Packages_THT:TO-220_Neutral123_Vertical_LargePads -> TO_SOT_Packages_THT:TO-92_Inline_Narrow_Oval
- R1, R9: value 150R -> R
- R10: value 20k -> 60k
- R11: value 150R -> 0.1R; footprint Resistors_ThroughHole:Resistor_Horizontal_RM7mm -> Resistors_ThroughHole:Resistor_Vertical_RM5mm
- R12: value 20k -> 0.1R; footprint Resistors_ThroughHole:Resistor_Horizontal_RM7mm -> Resistors_ThroughHole:Resistor_Vertical_RM5mm
- R13: value R -> 0.1R; footprint Resistors_ThroughHole:Resistor_Horizontal_RM7mm -> Resistors_ThroughHole:Resistor_Vertical_RM5mm
- R14: value 100k -> 0.1R; footprint Resistors_ThroughHole:Resistor_Horizontal_RM7mm -> Resistors_ThroughHole:Resistor_Vertical_RM5mm
- R15: value 68k -> 0.1R; footprint Resistors_ThroughHole:Resistor_Horizontal_RM7mm -> Resistors_ThroughHole:Resistor_Vertical_RM5mm
- R16, R2, R5: value 100k -> R
- R17, R3, R6, R8: value 68k -> R
- R18: value 150R -> 10k
- R19, R4: value 20k -> 220R
- R7: value 100k -> 220R
- U1: value LTV-817 -> LM358; footprint Housings_DIP:DIP-4_W7.62mm_LongPads -> Housings_DIP:DIP-8_W7.62mm_LongPads
- moved P2 374.5 mm to (80.0, 40.6), turned to 0 degrees
- moved R11 355.6 mm to (63.5, 63.5), turned to 90 degrees
- moved JP1 294.8 mm to (123.2, 77.5)
- moved C1 294.7 mm to (63.5, 48.3), turned to 270 degrees
- moved R9 285.6 mm to (132.1, 58.4), turned to 180 degrees
- moved C3 284.6 mm to (88.9, 48.3)
- moved P5 278.2 mm to (110.5, 40.6), turned to 0 degrees
- moved C4 276.9 mm to (101.6, 48.3)
- moved C5 263.3 mm to (114.3, 48.3), turned to 270 degrees
- moved R13 255.0 mm to (101.6, 63.5), turned to 90 degrees
- moved R18 254.0 mm to (179.1, 81.3), turned to 0 degrees
- moved C7 240.2 mm to (120.7, 45.7), turned to 90 degrees
- moved C6 237.7 mm to (128.3, 45.7), turned to 90 degrees
- moved D1 232.9 mm to (78.7, 27.9), turned to 0 degrees
- moved P20 229.0 mm to (53.3, 53.3), turned to 270 degrees
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Connections:
- C1 pad 1: +3V3 -> +36V
- C1 pad 2: GNDD -> GNDPWR
- C2 pad 1: +3V3 -> +36V
- C2 pad 2: GNDD -> GNDPWR
- C3 pad 1: +9V -> +36V
- C3 pad 2: GNDA -> GNDPWR
- C4 pad 1: +3V3 -> +36V
- C4 pad 2: GNDA -> GNDPWR
- C5 pad 1: Net-(1k1-Pad2) -> +36V
- C5 pad 2: GNDA -> GNDPWR
- C6 pad 1: +3V3 -> +36V
- C6 pad 2: GNDA -> GNDPWR
- C7 pad 1: +3V3 -> +36V
- C7 pad 2: GNDA -> GNDPWR
- D1 pad 1: Net-(D1-Pad1) -> +36V
- D2 pad 1: Net-(D2-Pad1) -> +36V
- D2 pad 2: Net-(D2-Pad2) -> Net-(D1-Pad2)
- D3 pad 1: Net-(D3-Pad1) -> +36V
- D4 pad 1: Net-(D4-Pad1) -> +36V
- D4 pad 2: Net-(D4-Pad2) -> Net-(D3-Pad2)
- D5 pad 1: Net-(D5-Pad1) -> +36V
- D6 pad 1: Net-(D6-Pad1) -> Net-(C10-Pad1)
- D6 pad 2: Net-(D6-Pad2) -> GNDPWR
- D7 pad 2: Net-(D7-Pad2) -> GNDPWR
- JP1 pad 1: GNDD -> Net-(JP1-Pad1)
- JP1 pad 2: /ts1 -> Net-(C12-Pad1)
- JP2 pad 1: GNDD -> Net-(JP2-Pad1)
- JP2 pad 2: /ts2 -> Net-(C18-Pad1)
- P1 pad 1: GNDPWR -> +36V
- P1 pad 2: +36V -> Net-(D1-Pad2)
- P10 pad 1: (no net) -> +9V
- P11 pad 1: +3V3 -> +9V
- P11 pad 2: GNDA -> Net-(P10-Pad2)
- P12 pad 1: (no net) -> +9V
- P13 pad 1: Net-(D3-Pad1) -> Net-(P13-Pad1)
- P13 pad 2: Net-(D3-Pad2) -> GNDA
- P2 pad 1: GNDPWR -> +36V
- P2 pad 2: +48V -> Net-(D1-Pad2)
- P20 pad 1: GNDPWR -> +36V
- P20 pad 2: +36V -> GNDPWR
- P3 pad 1: Net-(D2-Pad1) -> +36V
- P3 pad 2: Net-(D2-Pad2) -> Net-(D3-Pad2)
- P4 pad 1: GNDD -> +36V
- P4 pad 2: +12V -> Net-(D3-Pad2)
- P5 pad 1: GNDA -> +36V
- P5 pad 2: +9V -> Net-(D5-Pad2)
- P6 pad 1: Net-(D1-Pad2) -> Net-(P6-Pad1)
- P6 pad 2: Net-(D5-Pad2) -> Net-(P6-Pad2)
- P7 pad 1: (no net) -> Net-(P7-Pad1)
- P8 pad 1: Net-(IC1-Pad1) -> Net-(P8-Pad1)
- P9 pad 1: (no net) -> +9V
- Q1 pad 1: GNDPWR -> Net-(P6-Pad1)
- Q1 pad 2: Net-(Q1-Pad2) -> Net-(JP1-Pad1)
- Q1 pad 3: Net-(Q1-Pad3) -> GNDPWR
- Q2 pad 1: Net-(D2-Pad2) -> Net-(JP1-Pad1)
- Q2 pad 2: Net-(Q1-Pad3) -> Net-(Q2-Pad2)
- Q2 pad 3: GNDPWR -> Net-(D5-Pad2)
- Q3 pad 1: GNDPWR -> Net-(JP1-Pad1)
- Q3 pad 2: Net-(Q3-Pad2) -> Net-(Q2-Pad2)
- Q3 pad 3: Net-(Q3-Pad3) -> Net-(D3-Pad2)
- Q4 pad 1: GNDPWR -> +36V
- Q4 pad 3: Net-(Q4-Pad3) -> Net-(D7-Pad1)
- Q5 pad 1: Net-(D3-Pad2) -> Net-(JP1-Pad1)
- Q5 pad 2: Net-(Q3-Pad3) -> Net-(Q2-Pad2)
- Q5 pad 3: GNDPWR -> Net-(D1-Pad2)
- Q6 pad 1: Net-(D4-Pad2) -> Net-(P10-Pad2)
- Q6 pad 2: Net-(Q4-Pad3) -> Net-(JP2-Pad1)
- Q6 pad 3: GNDPWR -> GNDA
- R1 pad 1: GNDA -> Net-(Q4-Pad2)
- R10 pad 1: GNDPWR -> GNDA
- R10 pad 2: Net-(Q3-Pad3) -> Net-(JP2-Pad1)
- R11 pad 1: GNDA -> Net-(Q2-Pad2)
- R11 pad 2: Net-(R11-Pad2) -> GNDPWR
- R12 pad 1: GNDPWR -> Net-(Q2-Pad2)
- R12 pad 2: Net-(Q4-Pad3) -> GNDPWR
- R13 pad 1: Net-(IC1-Pad1) -> Net-(Q2-Pad2)
- R13 pad 2: +3V3 -> GNDPWR
- R14 pad 1: Net-(Q7-Pad2) -> Net-(Q2-Pad2)
- R14 pad 2: Net-(D7-Pad1) -> GNDPWR
- R15 pad 1: Net-(Q7-Pad3) -> Net-(Q2-Pad2)
- R15 pad 2: Net-(D7-Pad1) -> GNDPWR
- R16 pad 1: Net-(Q8-Pad2) -> +36V
- R16 pad 2: Net-(D8-Pad1) -> Net-(C12-Pad1)
- R17 pad 1: Net-(Q10-Pad2) -> Net-(JP1-Pad1)
- R17 pad 2: Net-(D8-Pad1) -> GNDPWR
- R18 pad 1: GNDA -> +9V
- R18 pad 2: Net-(R18-Pad2) -> Net-(C18-Pad1)
- R19 pad 1: GNDPWR -> Net-(JP2-Pad1)
- R19 pad 2: Net-(Q7-Pad3) -> Net-(P13-Pad1)
- R2 pad 1: Net-(Q1-Pad2) -> +36V
- R2 pad 2: Net-(D2-Pad1) -> Net-(C10-Pad1)
- R3 pad 1: Net-(Q1-Pad3) -> +36V
- R3 pad 2: Net-(D2-Pad1) -> Net-(C10-Pad1)
- R4 pad 1: GNDPWR -> Net-(P6-Pad2)
- R4 pad 2: Net-(Q1-Pad3) -> +5V
- R5 pad 1: Net-(Q3-Pad2) -> Net-(C10-Pad1)
- R5 pad 2: Net-(D3-Pad1) -> Net-(R1-Pad2)
- R6 pad 1: Net-(Q3-Pad3) -> GNDPWR
- R6 pad 2: Net-(D3-Pad1) -> Net-(R1-Pad2)
- R7 pad 1: Net-(Q4-Pad2) -> Net-(P7-Pad1)
- R7 pad 2: Net-(D4-Pad1) -> +5V
- R8 pad 1: Net-(Q4-Pad3) -> Net-(Q4-Pad2)
- R8 pad 2: Net-(D4-Pad1) -> Net-(C13-Pad1)
- R9 pad 1: GNDA -> Net-(C14-Pad1)
- R9 pad 2: Net-(R9-Pad2) -> Net-(Q2-Pad2)
- U1 pad 1: (no net) -> Net-(Q4-Pad2)
- U1 pad 2: Net-(R1-Pad2) -> Net-(C13-Pad1)
- U1 pad 3: GNDPWR -> Net-(R1-Pad2)
- U1 pad 4: Net-(Q1-Pad2) -> GNDPWR
Routing:
- net /ts1: track 81.6 -> 0.00 mm
- net (no net): track 78.1 -> 0.00 mm
- net /ts2: track 67.3 -> 0.00 mm
- net /ts6: track 56.2 -> 0.00 mm
- net /ts9: track 55.9 -> 0.00 mm
- net /ts8: track 43.4 -> 0.00 mm
- net +3V3: track 42.3 -> 0.00 mm
- net /ts3: track 32.7 -> 0.00 mm
- net /ts4: track 29.8 -> 0.00 mm
- net /ts5: track 27.8 -> 0.00 mm
- net +9V: track 21.6 -> 0.00 mm
- net Net-(1k1-Pad2): track 11.4 -> 0.00 mm
- net Net-(D15-Pad2): track 11.2 -> 0.00 mm
- net Net-(D9-Pad2): track 11.2 -> 0.00 mm
- net Net-(D6-Pad2): track 10.9 -> 0.00 mm
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