File: power_switch.sch (KiCad schematic (older format))
At the start: 52 parts, among them P1 CONN_2, P10 CONN_2, P11 CONN_2, P12 CONN_2, P13 CONN_02X01, P2 CONN_2, P20 CONN_2, P3 CONN_2, P4 CONN_2, P5 CONN_2, P6 CONN_2, P7 CONN_02X01, P8 CONN_02X01, P9 CONN_2, Q1 IRF9540, Q2 IRF9540, Q3 IRF9540, Q4 Q_NMOS_DGS, Q5 IRF9540, U1 LM358

Commit message: corrected switching transistor pins order
Parts:
- removed C8: 10uF, Capacitors_ThroughHole:CP_Radial_D4.0mm_P2.00mm, symbol CP
- removed D6, D8: 5v6, Diodes_ThroughHole:D_DO-35_SOD27_P7.62mm_Horizontal, symbol D_Zener
- removed R2: R, Resistors_ThroughHole:R_Axial_DIN0207_L6.3mm_D2.5mm_P7.62mm_Horizontal, symbol R
- added C7: 100n, Capacitors_ThroughHole:C_Disc_D3_P2.5, symbol C
- added U2: LM7805, Transistors_TO-220:TO-220_L78XX, symbol LM7805
- C1, C2, C3, C4, C5: footprint Capacitors_ThroughHole:C_Radial_D10_L20_P7.5 -> Capacitors_Elko_ThroughHole:Elko_vert_20x10mm_RM5
- C14: footprint Capacitors_ThroughHole:C_Radial_D8_L11.5_P3.5 -> Capacitors_Elko_ThroughHole:Elko_vert_11.2x6.3mm_RM2.5
- C6: footprint Capacitors_ThroughHole:CP_Radial_D6.3mm_P2.50mm -> Capacitors_Elko_ThroughHole:Elko_vert_11.2x6.3mm_RM2.5
- Q1, Q2, Q3, Q5: footprint TO_SOT_Packages_THT:TO-220_Neutral123_Vertical_LargePads -> Transistors_TO-220:TO-220_Neutral123_Vertical_LargePads_wide; symbol Q_NJFET_GSD -> Q_NJFET_GDS
- R11, R12, R13, R14, R15: footprint Resistors_ThroughHole:R_Axial_DIN0411_L9.9mm_D3.6mm_P5.08mm_Vertical -> Resistors_ThroughHole:Resistor_Cement_KOA-BGR-3N
Connections:
- net labels added: +12V
Other:
- moved on the sheet: C10, P7, Q4, R19, R20, R5, R7, RV1
